File: washing-machine.sch (EAGLE design)
At the start: 57 parts, among them IC1 MEGA8-P, IC2 7805TV, K1 ZNS5106, K2 ZNS5106, K3 ZNS5106, Q2 BC547, Q3 BC547, Q4 BC547, Q5 BC547, Q6 BC547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

Commit message: Minor modifications in the layout
Parts:
- added JP7: (no value), pinhead:PINHD-1X1
- added JP8: (no value), pinhead:PINHD-1X2
- JP2: device pinhead:PINHD-1X2 -> pinhead:PINHD-1X3
Connections:
- new net N$31: IC1.PD1(TXD), JP8.2
- new net N$38: IC1.PD0(RXD), JP8.1
- new net N$39: IC1.PC1(ADC1), JP7.1
- net +5V: now also JP2.3
Changed lines of the file:
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@@
 <part name="X2" library="con-ptr500" deviceset="AK500/3" device=""/>
 <part name="X3" library="con-ptr500" deviceset="AK500/3" device=""/>
-<part name="JP2" library="pinhead" deviceset="PINHD-1X2" device=""/>
+<part name="JP2" library="pinhead" deviceset="PINHD-1X3" device=""/>
 <part name="P+7" library="supply1" deviceset="+12V" device=""/>
 <part name="GND3" library="supply1" deviceset="GND" device=""/>
@@
 <part name="JP6" library="pinhead" deviceset="PINHD-1X6" device=""/>
 <part name="P+14" library="supply1" deviceset="+5V" device=""/>
+<part name="JP7" library="pinhead" deviceset="PINHD-1X1" device=""/>
+<part name="JP8" library="pinhead" deviceset="PINHD-1X2" device=""/>
+<part name="P+1" library="supply1" deviceset="+5V" device=""/>
 </parts>
 <sheets>
@@
 <instance part="X3" gate="-2" x="307.34" y="127" rot="R180"/>
 <instance part="X3" gate="-3" x="307.34" y="121.92" rot="R180"/>
-<instance part="JP2" gate="G$1" x="-40.64" y="78.74"/>
+<instance part="JP2" gate="A" x="-40.64" y="78.74"/>
 <instance part="P+7" gate="1" x="-50.8" y="83.82"/>
 <instance part="GND3" gate="1" x="-50.8" y="76.2"/>
@@
 <instance part="JP6" gate="A" x="373.38" y="45.72"/>
 <instance part="P+14" gate="1" x="370.84" y="63.5"/>
+<instance part="JP7" gate="G$1" x="99.06" y="71.12"/>
+<instance part="JP8" gate="G$1" x="71.12" y="50.8"/>
+<instance part="P+1" gate="1" x="-40.64" y="68.58" rot="R270"/>
 </instances>
 <busses>
@@
 </segment>
 <segment>
-<pinref part="JP2" gate="G$1" pin="1"/>
+<pinref part="JP2" gate="A" pin="1"/>
 <pinref part="P+7" gate="1" pin="+12V"/>
 <wire x1="-50.8" y1="81.28" x2="-43.18" y2="81.28" width="0.1524" layer="91"/>
@@
 <pinref part="P+14" gate="1" pin="+5V"/>
 <wire x1="370.84" y1="60.96" x2="370.84" y2="53.34" width="0.1524" layer="91"/>
+</segment>
+<segment>
+<pinref part="P+1" gate="1" pin="+5V"/>
+<pinref part="JP2" gate="A" pin="3"/>
+<wire x1="-43.18" y1="68.58" x2="-43.18" y2="76.2" width="0.1524" layer="91"/>
 </segment>
 </net>
@@
 </segment>
 <segment>
-<pinref part="JP2" gate="G$1" pin="2"/>
+<pinref part="JP2" gate="A" pin="2"/>
 <pinref part="GND3" gate="1" pin="GND"/>
 <wire x1="-50.8" y1="78.74" x2="-43.18" y2="78.74" width="0.1524" layer="91"/>
@@
 </segment>
 </net>
+<net name="N$31" class="0">
+<segment>
+<pinref part="IC1" gate="G$1" pin="PD1(TXD)"/>
+<pinref part="JP8" gate="G$1" pin="2"/>
+<wire x1="58.42" y1="48.26" x2="68.58" y2="48.26" width="0.1524" layer="91"/>
+<wire x1="68.58" y1="48.26" x2="68.58" y2="50.8" width="0.1524" layer="91"/>
+</segment>
+</net>
+<net name="N$38" class="0">
+<segment>
+<pinref part="IC1" gate="G$1" pin="PD0(RXD)"/>
+<wire x1="58.42" y1="50.8" x2="66.04" y2="50.8" width="0.1524" layer="91"/>
+<wire x1="66.04" y1="50.8" x2="66.04" y2="53.34" width="0.1524" layer="91"/>
+<pinref part="JP8" gate="G$1" pin="1"/>
+<wire x1="66.04" y1="53.34" x2="68.58" y2="53.34" width="0.1524" layer="91"/>
+</segment>
+</net>
+<net name="N$39" class="0">
+<segment>
+<pinref part="IC1" gate="G$1" pin="PC1(ADC1)"/>
+<pinref part="JP7" gate="G$1" pin="1"/>
+<wire x1="58.42" y1="71.12" x2="96.52" y2="71.12" width="0.1524" layer="91"/>
+</segment>
+</net>
